Commit message: added gps data in ekf

File: src/description/urdf/robot_base.xacro (robot description, xacro)
@@ -14,5 +14,5 @@
           <box size="${base_length} ${base_width} ${base_height}"/>
         </geometry>
-        <origin xyz="0 0 ${base_height/2}" rpy="0 0 0"/>
+        <origin xyz="0 0 ${base_height/2 + wheel_radius}" rpy="0 0 0"/>
         <material name="body_color">
           <color rgba="0.15 0.15 0.18 1"/>
@@ -23,9 +23,9 @@
           <box size="${base_length} ${base_width} ${base_height}"/>
         </geometry>
-        <origin xyz="0 0 ${base_height/2}" rpy="0 0 0"/>
+        <origin xyz="0 0 ${base_height/2 + wheel_radius}" rpy="0 0 0"/>
       </collision>
       <inertial>
         <mass value="10.0"/>
-        <origin xyz="0 0 ${base_height/2}"/>
+        <origin xyz="0 0 ${base_height/2 + wheel_radius}"/>
         <inertia ixx="0.2" iyy="0.2" izz="0.2" ixy="0" ixz="0" iyz="0"/>
       </inertial>

File: src/description/urdf/robot_sensors.xacro (robot description, xacro)
@@ -14,4 +14,21 @@
         <update_rate>5</update_rate>
         <topic>/gps</topic>
+        <gz_frame_id>gps_link</gz_frame_id>
+        <navsat>
+          <position_sensing>
+            <horizontal>
+              <noise type="gaussian">
+                <mean>0</mean>
+                <stddev>0.000005</stddev>
+              </noise>
+            </horizontal>
+            <vertical>
+              <noise type="gaussian">
+                <mean>0</mean>
+                <stddev>0.000005</stddev>
+              </noise>
+            </vertical>
+          </position_sensing>
+        </navsat>
       </sensor>
     </gazebo>
