Commit message: without encoders

File: src/description/urdf/robot_base.xacro (robot description, xacro)
@@ -2,11 +2,25 @@
 <robot xmlns:xacro="http://www.ros.org/wiki/xacro">
   <xacro:macro name="base">
-    <xacro:property name="base_length" value="0.5"/>
-    <xacro:property name="base_width" value="0.4"/>
-    <xacro:property name="base_height" value="0.2"/>
-    <xacro:property name="wheel_radius" value="0.075"/>
-    <xacro:property name="wheel_width" value="0.04"/>
-    <xacro:property name="wheel_x_offset" value="0.18"/>
-    <xacro:property name="wheel_y_offset" value="0.22"/>
+    <!-- ================= DIMENSIONS ================= -->
+    <xacro:property name="base_length"       value="0.55"/>
+    <xacro:property name="base_width"        value="0.48"/>
+    <xacro:property name="base_height"       value="0.29"/>
+    <xacro:property name="ground_clearance"  value="0.09"/>
+    <xacro:property name="base_mass"         value="28.0"/>
+    <!-- Wheel diameter = 32 cm -> radius = 16 cm (0.16 m) -->
+    <xacro:property name="wheel_radius"      value="0.16"/>
+    <xacro:property name="wheel_width"       value="0.06"/>
+    <xacro:property name="wheel_mass"        value="1.2"/>
+    <!-- Drive wheels position (rear) -->
+    <xacro:property name="wheel_x_offset"    value="-0.15"/>
+    <xacro:property name="wheel_y_offset"    value="0.27"/> <!-- Separation = 0.54 m -->
+    <!-- Front castor (touches ground at z = 0) -->
+    <xacro:property name="castor_radius"     value="0.039"/>
+    <xacro:property name="castor_x_offset"   value="0.20"/>
+    <xacro:property name="castor_strut_height"
+                    value="${ground_clearance - 2 * castor_radius}"/>
+    <!-- Base box center z relative to ground (z=0): 0.09 + 0.29/2 = 0.235m -->
+    <xacro:property name="base_z_center"     value="${ground_clearance + base_height / 2}"/>
+    <!-- ================= BASE LINK ================= -->
     <link name="base_link">
       <visual>
@@ -14,5 +28,5 @@
           <box size="${base_length} ${base_width} ${base_height}"/>
         </geometry>
-        <origin xyz="0 0 ${base_height/2 + wheel_radius}" rpy="0 0 0"/>
+        <origin xyz="0 0 ${base_z_center}" rpy="0 0 0"/>
         <material name="body_color">
           <color rgba="0.15 0.15 0.18 1"/>
@@ -23,10 +37,11 @@
           <box size="${base_length} ${base_width} ${base_height}"/>
         </geometry>
-        <origin xyz="0 0 ${base_height/2 + wheel_radius}" rpy="0 0 0"/>
-      </collision>
-      <inertial>
-        <mass value="10.0"/>
-        <origin xyz="0 0 ${base_height/2 + wheel_radius}"/>
-        <inertia ixx="0.2" iyy="0.2" izz="0.2" ixy="0" ixz="0" iyz="0"/>
+        <origin xyz="0 0 ${base_z_center}" rpy="0 0 0"/>
+      </collision>
+      <inertial>
+        <mass value="${base_mass}"/>
+        <origin xyz="-0.069 0.0 ${base_z_center}"/>
+        <inertia ixx="1.708" iyy="2.802" izz="1.732"
+                 ixy="0" ixz="0" iyz="0"/>
       </inertial>
     </link>
@@ -34,172 +49,5 @@
       <self_collide>false</self_collide>
     </gazebo>
-    <link name="imu_link">
-      <visual>
-        <geometry>
-          <box size="0.03 0.03 0.02"/>
-        </geometry>
-        <origin xyz="0 0 0"/>
-        <material name="orange">
-          <color rgba="1 0.5 0 1"/>
-        </material>
-      </visual>
-    </link>
-    <joint name="imu_joint" type="fixed">
-      <parent link="base_link"/>
-      <child link="imu_link"/>
-      <origin xyz="0 0 0.15"/>
-    </joint>
-    <link name="gps_link">
-      <visual>
-        <geometry>
-          <box size="0.03 0.03 0.02"/>
-        </geometry>
-        <origin xyz="0 0 0"/>
-        <material name="white">
-          <color rgba="1 1 1 1"/>
-        </material>
-      </visual>
-    </link>
-    <joint name="gps_joint" type="fixed">
-      <parent link="base_link"/>
-      <child link="gps_link"/>
-      <origin xyz="0 0 0.2"/>
-    </joint>
-    <link name="lidar_link">
-      <visual>
-        <geometry>
-          <cylinder radius="0.04" length="0.05"/>
-        </geometry>
-        <origin xyz="0 0 0"/>
-        <material name="gray">
-          <color rgba="0.6 0.6 0.6 1.0"/>
-        </material>
-      </visual>
-      <collision>
-        <geometry>
-          <cylinder radius="0.04" length="0.05"/>
-        </geometry>
-        <origin xyz="0 0 0"/>
-      </collision>
-    </link>
-    <joint name="lidar_joint" type="fixed">
-      <parent link="base_link"/>
-      <child link="lidar_link"/>
-      <origin xyz="0.22 0 0.22"/>
-    </joint>
-    <!-- ================= PAN LINK ================= -->
-<link name="pan_link">
-  <visual>
-    <geometry>
-      <cylinder radius="0.05" length="0.02"/>
-    </geometry>
-    <material name="red">
-      <color rgba="1 0 0 1"/>
-    </material>
-  </visual>
-  <collision>
-    <geometry>
-      <cylinder radius="0.05" length="0.02"/>
-    </geometry>
-  </collision>
-  <inertial>
-    <mass value="0.5"/>
-    <origin xyz="0 0 0"/>
-    <inertia ixx="0.01" iyy="0.01" izz="0.01"
-             ixy="0" ixz="0" iyz="0"/>
-  </inertial>
-</link>
-<joint name="pan_joint" type="revolute">
-  <parent link="base_link"/>
-  <child link="pan_link"/>
-  <origin xyz="0.12 0 0.21"/>
-  <axis xyz="0 0 1"/>
-  <limit lower="-3.14" upper="3.14" effort="5" velocity="1"/>
-  <dynamics damping="0.1" friction="0.1"/>
-</joint>
-<!-- ================= TILT LINK ================= -->
-<link name="tilt_link">
-  <visual>
-    <geometry>
-      <box size="0.04 0.04 0.02"/>
-    </geometry>
-    <material name="black">
-      <color rgba="0.1 0.1 0.1 1"/>
-    </material>
-  </visual>
-  <collision>
-    <geometry>
-      <box size="0.04 0.04 0.02"/>
-    </geometry>
-  </collision>
-  <inertial>
-    <mass value="0.3"/>
-    <origin xyz="0 0 0"/>
-    <inertia ixx="0.005" iyy="0.005" izz="0.005"
-             ixy="0" ixz="0" iyz="0"/>
-  </inertial>
-</link>
-<joint name="tilt_base_joint" type="revolute">
-  <parent link="pan_link"/>
-  <child link="tilt_link"/>
-  <origin xyz="0 0 0.05"/>
-  <axis xyz="0 1 0"/>
-  <limit lower="-1.57" upper="1.57" effort="5" velocity="1"/>
-  <dynamics damping="0.1" friction="0.1"/>
-</joint>
-<!-- ================= TURRET CAMERA ================= -->
-<link name="turret_camera_link">
-  <visual>
-    <geometry>
-      <box size="0.05 0.05 0.05"/>
-    </geometry>
-    <material name="Red">
-      <color rgba="1 0 0 1"/>
-    </material>
-  </visual>
-  <collision>
-    <geometry>
-      <box size="0.05 0.05 0.05"/>
-    </geometry>
-  </collision>
-  <inertial>
-    <mass value="0.3"/>
-    <origin xyz="0 0 0"/>
-    <inertia ixx="0.005" iyy="0.005" izz="0.005"
-             ixy="0" ixz="0" iyz="0"/>
-  </inertial>
-</link>
-<joint name="turret_camera_joint" type="fixed">
-  <parent link="tilt_link"/>
-  <child link="turret_camera_link"/>
-  <origin xyz="0 0 0.03"/>
-</joint>
-<!-- ================= LANE CAMERA ================= -->
-<link name="camera_link">
-  <visual>
-    <geometry>
-      <box size="0.05 0.05 0.05"/>
-    </geometry>
-    <material name="blue">
-      <color rgba="0 0 1 1"/>
-    </material>
-  </visual>
-  <collision>
-    <geometry>
-      <box size="0.05 0.05 0.05"/>
-    </geometry>
-  </collision>
-  <inertial>
-    <mass value="0.3"/>
-    <origin xyz="0 0 0"/>
-    <inertia ixx="0.005" iyy="0.005" izz="0.005"
-             ixy="0" ixz="0" iyz="0"/>
-  </inertial>
-</link>
-<joint name="camera_joint" type="fixed">
-  <parent link="base_link"/>
-  <child link="camera_link"/>
-  <origin xyz="0.15 0 1" rpy="0 0.25 0"/> <!-- chcanged camera and turret positions-->
-</joint>
+    <!-- ================= DRIVE WHEEL MACRO ================= -->
     <xacro:macro name="wheel" params="name x y">
       <link name="${name}_link">
@@ -209,5 +57,5 @@
             <cylinder radius="${wheel_radius}" length="${wheel_width}"/>
           </geometry>
-          <material name="black">
+          <material name="wheel_black">
             <color rgba="0.05 0.05 0.05 1"/>
           </material>
@@ -220,5 +68,5 @@
         </collision>
         <inertial>
-          <mass value="1.0"/>
+          <mass value="${wheel_mass}"/>
           <origin xyz="0 0 0"/>
           <inertia ixx="0.01" iyy="0.01" izz="0.005" ixy="0" ixz="0" iyz="0"/>
@@ -232,16 +80,245 @@
       </joint>
     </xacro:macro>
-    <xacro:wheel name="front_left_wheel"
+    <!-- Two drive wheels (rear) -->
+    <xacro:wheel name="left_wheel"
                  x="${wheel_x_offset}"
                  y="${wheel_y_offset}"/>
-    <xacro:wheel name="rear_left_wheel"
-                 x="-${wheel_x_offset}"
-                 y="${wheel_y_offset}"/>
-    <xacro:wheel name="front_right_wheel"
+    <xacro:wheel name="right_wheel"
                  x="${wheel_x_offset}"
                  y="-${wheel_y_offset}"/>
-    <xacro:wheel name="rear_right_wheel"
-                 x="-${wheel_x_offset}"
-                 y="-${wheel_y_offset}"/>
+    <!-- ================= CASTOR WHEEL (FRONT) ================= -->
+    <!-- Vertical strut connecting chassis bottom to castor ball -->
+    <link name="castor_strut_link">
+      <visual>
+        <geometry>
+          <cylinder radius="0.012" length="${castor_strut_height}"/>
+        </geometry>
+        <origin xyz="0 0 ${-castor_strut_height/2}"/>
+        <material name="strut_gray">
+          <color rgba="0.4 0.4 0.4 1"/>
+        </material>
+      </visual>
+      <collision>
+        <geometry>
+          <cylinder radius="0.012" length="${castor_strut_height}"/>
+        </geometry>
+        <origin xyz="0 0 ${-castor_strut_height/2}"/>
+      </collision>
+      <inertial>
+        <mass value="0.1"/>
+        <origin xyz="0 0 0"/>
+        <inertia ixx="0.001" iyy="0.001" izz="0.001" ixy="0" ixz="0" iyz="0"/>
+      </inertial>
+    </link>
+    <joint name="castor_strut_joint" type="fixed">
+      <parent link="base_link"/>
+      <child link="castor_strut_link"/>
+      <origin xyz="${castor_x_offset} 0 ${ground_clearance}"/>
+    </joint>
+    <!-- Castor ball – touches ground at z=0 -->
+    <link name="castor_wheel_link">
+      <visual>
+        <geometry>
+          <sphere radius="${castor_radius}"/>
+        </geometry>
+        <material name="castor_gray">
+          <color rgba="0.6 0.6 0.6 1"/>
+        </material>
+      </visual>
+      <collision>
+        <geometry>
+          <sphere radius="${castor_radius}"/>
+        </geometry>
+      </collision>
+      <inertial>
+        <mass value="0.3"/>
+        <origin xyz="0 0 0"/>
+        <inertia ixx="0.001" iyy="0.001" izz="0.001" ixy="0" ixz="0" iyz="0"/>
+      </inertial>
+    </link>
+    <joint name="castor_wheel_joint" type="fixed">
+      <parent link="castor_strut_link"/>
+      <child link="castor_wheel_link"/>
+      <origin xyz="0 0 ${-castor_strut_height - castor_radius}"/>
+    </joint>
+    <!-- Zero friction so castor slides freely in Gazebo -->
+    <gazebo reference="castor_wheel_link">
+      <mu1>0.0</mu1>
+      <mu2>0.0</mu2>
+      <slip1>1.0</slip1>
+      <slip2>1.0</slip2>
+      <fdir1>0 0 1</fdir1>
+    </gazebo>
+    <!-- ================= IMU ================= -->
+    <link name="imu_link">
+      <visual>
+        <geometry>
+          <box size="0.03 0.03 0.02"/>
+        </geometry>
+        <origin xyz="0 0 0"/>
+        <material name="orange">
+          <color rgba="1 0.5 0 1"/>
+        </material>
+      </visual>
+    </link>
+    <joint name="imu_joint" type="fixed">
+      <parent link="base_link"/>
+      <child link="imu_link"/>
+      <origin xyz="0 0 ${ground_clearance + base_height + 0.01}"/>
+    </joint>
+    <!-- ================= GPS ================= -->
+    <link name="gps_link">
+      <visual>
+        <geometry>
+          <box size="0.03 0.03 0.02"/>
+        </geometry>
+        <origin xyz="0 0 0"/>
+        <material name="white">
+          <color rgba="1 1 1 1"/>
+        </material>
+      </visual>
+    </link>
+    <joint name="gps_joint" type="fixed">
+      <parent link="base_link"/>
+      <child link="gps_link"/>
+      <origin xyz="0 0 ${ground_clearance + base_height + 0.05}"/>
+    </joint>
+    <!-- ================= LIDAR (laser_link) ================= -->
+    <link name="laser_link">
+      <visual>
+        <geometry>
+          <cylinder radius="0.04" length="0.05"/>
+        </geometry>
+        <origin xyz="0 0 0"/>
+        <material name="gray">
+          <color rgba="0.6 0.6 0.6 1.0"/>
+        </material>
+      </visual>
+      <collision>
+        <geometry>
+          <cylinder radius="0.04" length="0.05"/>
+        </geometry>
+        <origin xyz="0 0 0"/>
+      </collision>
+    </link>
+    <joint name="laser_joint" type="fixed">
+      <parent link="base_link"/>
+      <child link="laser_link"/>
+      <origin xyz="0.22 0 ${ground_clearance + base_height + 0.03}" rpy="0 0 3.14159"/>
+    </joint>
+    <!-- ================= PAN LINK ================= -->
+    <link name="pan_link">
+      <visual>
+        <geometry>
+          <cylinder radius="0.05" length="0.02"/>
+        </geometry>
+        <material name="red">
+          <color rgba="1 0 0 1"/>
+        </material>
+      </visual>
+      <collision>
+        <geometry>
+          <cylinder radius="0.05" length="0.02"/>
+        </geometry>
+      </collision>
+      <inertial>
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
File: src/description/urdf/robot_control.xacro (robot description, xacro)
@@ -2,25 +2,16 @@
 <robot xmlns:xacro="http://www.ros.org/wiki/xacro">
 <xacro:macro name="control">
-  <ros2_control name="SkidSteerSystem" type="system">
+  <ros2_control name="DiffDriveSystem" type="system">
   <hardware>
     <plugin>gz_ros2_control/GazeboSimSystem</plugin>
   </hardware>
-  <!-- Wheels -->
-  <joint name="front_left_wheel_joint">
+  <!-- Left drive wheel -->
+  <joint name="left_wheel_joint">
     <command_interface name="velocity"/>
     <state_interface name="position"/>
     <state_interface name="velocity"/>
   </joint>
-  <joint name="rear_left_wheel_joint">
-    <command_interface name="velocity"/>
-    <state_interface name="position"/>
-    <state_interface name="velocity"/>
-  </joint>
-  <joint name="front_right_wheel_joint">
-    <command_interface name="velocity"/>
-    <state_interface name="position"/>
-    <state_interface name="velocity"/>
-  </joint>
-  <joint name="rear_right_wheel_joint">
+  <!-- Right drive wheel -->
+  <joint name="right_wheel_joint">
     <command_interface name="velocity"/>
     <state_interface name="position"/>

File: src/description/urdf/robot_real.urdf.xacro (robot description, xacro)
@@ -1,19 +1,89 @@
 <?xml version="1.0"?>
 <robot name="mercury" xmlns:xacro="http://www.ros.org/wiki/xacro">
-  <!-- ================= BASE ================= -->
+  <!-- ================= BASE CHASSIS ================= -->
+  <!-- Dimensions: length=55cm (0.55m), width=48cm (0.48m), height=29cm (0.29m) -->
+  <!-- Ground clearance: 9cm (0.09m) -->
+  <!-- Center of chassis box z = 0.09 + (0.29 / 2) = 0.235m -->
   <link name="base_link">
     <visual>
       <geometry>
-        <box size="0.4 0.3 0.1"/>
+        <box size="0.55 0.48 0.29"/>
       </geometry>
-      <origin xyz="0 0 0.05"/>
+      <origin xyz="0 0 0.235" rpy="0 0 0"/>
+      <material name="chassis_color">
+        <color rgba="0.15 0.15 0.18 1.0"/>
+      </material>
     </visual>
   </link>
-  <!-- ================= LIDAR ================= -->
+  <!-- ================= LEFT DRIVE WHEEL ================= -->
+  <!-- Diameter = 32cm -> radius = 16cm (0.16m), width = 6cm (0.06m) -->
+  <!-- Wheel center z = 0.16m (touches ground at z=0) -->
+  <!-- Separation = 54cm (0.54m) -> y = +0.27m -->
+  <!-- Note: joint type is "fixed" because there are no physical wheel encoders. -->
+  <!-- This allows robot_state_publisher to broadcast the static TF without waiting for encoder /joint_states -->
+  <link name="left_wheel_link">
+    <visual>
+      <origin xyz="0 0 0" rpy="1.5708 0 0"/>
+      <geometry>
+        <cylinder radius="0.16" length="0.06"/>
+      </geometry>
+      <material name="wheel_black">
+        <color rgba="0.05 0.05 0.05 1.0"/>
+      </material>
+    </visual>
+  </link>
+  <joint name="left_wheel_joint" type="fixed">
+    <parent link="base_link"/>
+    <child link="left_wheel_link"/>
+    <origin xyz="-0.15 0.27 0.16" rpy="0 0 0"/>
+  </joint>
+  <!-- ================= RIGHT DRIVE WHEEL ================= -->
+  <!-- Separation = 54cm (0.54m) -> y = -0.27m -->
+  <link name="right_wheel_link">
+    <visual>
+      <origin xyz="0 0 0" rpy="1.5708 0 0"/>
+      <geometry>
+        <cylinder radius="0.16" length="0.06"/>
+      </geometry>
+      <material name="wheel_black">
+        <color rgba="0.05 0.05 0.05 1.0"/>
+      </material>
+    </visual>
+  </link>
+  <joint name="right_wheel_joint" type="fixed">
+    <parent link="base_link"/>
+    <child link="right_wheel_link"/>
+    <origin xyz="-0.15 -0.27 0.16" rpy="0 0 0"/>
+  </joint>
+  <!-- ================= FRONT CASTOR WHEEL ================= -->
+  <!-- Castor radius = 3.9cm (0.039m), touches ground at z=0 (origin z = 0.039m) -->
+  <!-- Positioned at front: x = +0.20m, y = 0.0m -->
+  <link name="castor_wheel_link">
+    <visual>
+      <geometry>
+        <sphere radius="0.039"/>
+      </geometry>
+      <origin xyz="0 0 0" rpy="0 0 0"/>
+      <material name="castor_gray">
+        <color rgba="0.5 0.5 0.5 1.0"/>
+      </material>
+    </visual>
+  </link>
+  <joint name="castor_wheel_joint" type="fixed">
+    <parent link="base_link"/>
+    <child link="castor_wheel_link"/>
+    <origin xyz="0.20 0.0 0.039" rpy="0 0 0"/>
+  </joint>
+  <!-- ================= RPLIDAR (laser_link) ================= -->
+  <!-- Mounted on top-front of chassis: z = 0.09 + 0.29 + 0.03 = 0.41m -->
   <link name="laser_link">
     <visual>
       <geometry>
-        <cylinder length="0.05" radius="0.05"/>
+        <cylinder length="0.05" radius="0.04"/>
       </geometry>
+      <origin xyz="0 0 0" rpy="0 0 0"/>
+      <material name="lidar_red">
+        <color rgba="0.8 0.1 0.1 1.0"/>
+      </material>
     </visual>
   </link>
@@ -21,5 +91,41 @@
     <parent link="base_link"/>
     <child link="laser_link"/>
-    <origin xyz="0.2 0 0.15" rpy="0 0 3.14159"/>
+    <origin xyz="0.22 0.0 0.41" rpy="0 0 3.14159"/>
+  </joint>
+  <!-- ================= IMU FRAME ================= -->
+  <!-- Fixed frame for IMU (ESP32-S3 / RealSense) -->
+  <link name="imu_link">
+    <visual>
+      <geometry>
+        <box size="0.03 0.03 0.02"/>
+      </geometry>
+      <origin xyz="0 0 0" rpy="0 0 0"/>
+      <material name="imu_orange">
+        <color rgba="1.0 0.5 0.0 1.0"/>
+      </material>
+    </visual>
+  </link>
+  <joint name="imu_joint" type="fixed">
+    <parent link="base_link"/>
+    <child link="imu_link"/>
+    <origin xyz="0.0 0.0 0.39" rpy="0 0 0"/>
+  </joint>
+  <!-- ================= GPS FRAME ================= -->
+  <!-- Mounted on top: z = 0.43m -->
+  <link name="gps_link">
+    <visual>
+      <geometry>
+        <box size="0.04 0.04 0.02"/>
+      </geometry>
+      <origin xyz="0 0 0" rpy="0 0 0"/>
+      <material name="gps_white">
+        <color rgba="0.9 0.9 0.9 1.0"/>
+      </material>
+    </visual>
+  </link>
+  <joint name="gps_joint" type="fixed">
+    <parent link="base_link"/>
+    <child link="gps_link"/>
+    <origin xyz="0.0 0.0 0.43" rpy="0 0 0"/>
   </joint>
   <!-- ================= REALSENSE CAMERA BODY ================= -->
@@ -28,8 +134,7 @@
     <parent link="base_link"/>
     <child link="camera_link"/>
-    <!-- Adjust these values to your real mounting -->
-    <origin xyz="0.15 0 0.12" rpy="0 0 0"/>
+    <origin xyz="0.15 0.0 0.38" rpy="0 0 0"/>
   </joint>
-  <!-- ================= IMU FRAME ================= -->
+  <!-- ================= CAMERA IMU FRAMES ================= -->
   <link name="camera_imu_frame"/>
   <joint name="camera_imu_joint" type="fixed">
@@ -38,5 +143,4 @@
     <origin xyz="0 0 0" rpy="0 0 0"/>
   </joint>
-  <!-- ================= IMU OPTICAL FRAME ================= -->
   <!-- Optical frame rotation: X right, Y down, Z forward -->
   <link name="camera_imu_optical_frame"/>
@@ -44,22 +148,5 @@
     <parent link="camera_imu_frame"/>
     <child link="camera_imu_optical_frame"/>
-    <!-- Convert from ROS frame to optical frame -->
     <origin xyz="0 0 0" rpy="-1.5708 0 -1.5708"/>
   </joint>
-  <link name="gps_link">
-      <visual>
-        <geometry>
-          <box size="0.03 0.03 0.02"/>
-        </geometry>
-        <origin xyz="0 0 0"/>
-        <material name="white">
-          <color rgba="1 1 1 1"/>
-        </material>
-      </visual>
-    </link>
-    <joint name="gps_joint" type="fixed">
-      <parent link="base_link"/>
-      <child link="gps_link"/>
-      <origin xyz="0 0 0.2"/>
-    </joint>
 </robot>

File: src/description/urdf/robot_sensors.xacro (robot description, xacro)
@@ -33,5 +33,5 @@
       </sensor>
     </gazebo>
-    <gazebo reference="lidar_link">
+    <gazebo reference="laser_link">
       <sensor name="lidar_sensor" type="gpu_lidar">
         <always_on>true</always_on>
@@ -39,5 +39,5 @@
         <topic>/scan</topic>
         <visualize>true</visualize>
-        <gz_frame_id>lidar_link</gz_frame_id>
+        <gz_frame_id>laser_link</gz_frame_id>
         <lidar>
           <scan>
@@ -77,22 +77,22 @@
     </gazebo>
     <gazebo reference="turret_camera_link">
-  <sensor name="turret_camera_sensor" type="camera">
-    <always_on>true</always_on>
-    <update_rate>30</update_rate>
-    <topic>/turret_camera/image_raw</topic>
-    <camera>
-      <horizontal_fov>1.047</horizontal_fov>
-      <image>
-        <width>640</width>
-        <height>480</height>
-        <format>R8G8B8</format>
-      </image>
-      <clip>
-        <near>0.1</near>
-        <far>100</far>
-      </clip>
-    </camera>
-  </sensor>
-</gazebo>
+      <sensor name="turret_camera_sensor" type="camera">
+        <always_on>true</always_on>
+        <update_rate>30</update_rate>
+        <topic>/turret_camera/image_raw</topic>
+        <camera>
+          <horizontal_fov>1.047</horizontal_fov>
+          <image>
+            <width>640</width>
+            <height>480</height>
+            <format>R8G8B8</format>
+          </image>
+          <clip>
+            <near>0.1</near>
+            <far>100</far>
+          </clip>
+        </camera>
+      </sensor>
+    </gazebo>
   </xacro:macro>
 </robot>
