Commit message: fixed lidar orientation and added camera controls

File: src/description/urdf/robot_real.urdf.xacro (robot description, xacro)
@@ -21,5 +21,5 @@
     <parent link="base_link"/>
     <child link="laser_link"/>
-    <origin xyz="0.2 0 0.15" rpy="0 0 0"/>
+    <origin xyz="0.2 0 0.15" rpy="0 0 3.14159"/>
   </joint>
   <!-- ================= REALSENSE CAMERA BODY ================= -->
